File: FeatherCAN.sch (KiCad schematic (older format))
At the start: 31 parts, among them J1 Feather Long, J2 Feather Short, J3 Header, J4 PicoBlade, U1 DS3231MZ, U2 MCP2515-xST, U3 MCP2551-I-SN, U4 5V, Y1 16MHz

Commit message: gerbers and kitspcae
Parts:
- added D4: 40V 200mA, KiCad/Diode_SMD.pretty:D_0603_1608Metric, symbol Device:D_Small
- added TP1: RTC_BAT, KiCad/TestPoint.pretty:TestPoint_Pad_D2.5mm, symbol Connector:TestPoint
- JP3, JP4: footprint KiCad/Jumper.pretty:SolderJumper-2_P1.3mm_Bridged_RoundedPad1.0x1.5mm -> KiCad/Jumper.pretty:SolderJumper-2_P1.3mm_Open_RoundedPad1.0x1.5mm; symbol Jumper:SolderJumper_2_Bridged -> Jumper:SolderJumper_2_Open
- R1: Characteristics (none) -> 1%
Connections:
- net VIN: now also D4.2 (A); no longer C1.1, U4.3 (VI)
- net +BATT: now reaches BT1.1 (+), U1.6 (VBAT)
- net +BATT: now also TP1.1
- new net: C1.1, D4.1 (K), U4.3 (VI)
Other:
- note added: "250 mA! 10k charge current resistor on Feather if using LiPo = 100 mA"
- moved on the sheet: C2, D3, R5
Changed lines of the file:
@@
 Wire Wire Line
 	4350 2000 4350 2400
-Wire Wire Line
-	4650 1700 5100 1700
-$Comp
-L power:GND #PWR0103
-U 1 1 5E08A9F1
-P 5100 2400
-F 0 "#PWR0103" H 5100 2150 50  0001 C CNN
-F 1 "GND" H 5100 2250 50  0000 C CNN
-F 2 "" H 5100 2400 50  0001 C CNN
-F 3 "" H 5100 2400 50  0001 C CNN
-	1    5100 2400
-	1    0    0    -1
-$EndComp
-Connection ~ 5100 1700
 $Comp
 L Regulator_Linear:MCP1700-5002E_SOT23 U4
@@
 	1    0    0    -1
 $EndComp
-$Comp
-L Device:C C2
-U 1 1 5DA6480B
-P 5100 2050
-F 0 "C2" H 5215 2096 50  0000 L CNN
-F 1 "1uF" H 5215 2005 50  0000 L CNN
-F 2 "KiCad/Capacitor_SMD.pretty:C_0603_1608Metric" H 5138 1900 50  0001 C CNN
-F 3 "~" H 5100 2050 50  0001 C CNN
-F 4 "X5R 20V" H 5100 2050 50  0001 C CNN "Characteristics"
-	1    5100 2050
-	1    0    0    -1
-$EndComp
-Wire Wire Line
-	5100 1700 5100 1900
-Wire Wire Line
-	5100 2200 5100 2400
 $Comp
 L Interface_CAN_LIN:MCP2515-xST U2
@@
 Connection ~ 8050 2700
 $Comp
-L Device:R_Small R1
-U 1 1 5E14102C
-P 2100 5550
-F 0 "R1" H 2130 5570 50  0000 L CNN
-F 1 "120R" H 2130 5510 50  0000 L CNN
-F 2 "KiCad/Resistor_SMD.pretty:R_0603_1608Metric" H 2100 5550 50  0001 C CNN
-F 3 "" H 2100 5550 50  0001 C CNN
-F 4 "Rterm" H 1950 5550 50  0000 C CNN "Description"
-	1    2100 5550
-	1    0    0    -1
-$EndComp
-$Comp
 L Jumper:SolderJumper_2_Open JP1
 U 1 1 5E142196
@@
 $EndComp
 Wire Wire Line
-	5100 1700 5500 1700
-Wire Wire Line
-	6850 1900 6850 2400
+	5950 1900 5950 2400
 $Comp
 L power:GND #PWR0116
 U 1 1 5E08A9F4
-P 6850 2400
-F 0 "#PWR0116" H 6850 2150 50  0001 C CNN
-F 1 "GND" H 6850 2250 50  0000 C CNN
-F 2 "" H 6850 2400 50  0001 C CNN
-F 3 "" H 6850 2400 50  0001 C CNN
-	1    6850 2400
-	1    0    0    -1
-$EndComp
-Wire Wire Line
-	6850 1600 6850 1700
-Wire Wire Line
-	6850 1200 6850 1300
+P 5950 2400
+F 0 "#PWR0116" H 5950 2150 50  0001 C CNN
+F 1 "GND" H 5950 2250 50  0000 C CNN
+F 2 "" H 5950 2400 50  0001 C CNN
+F 3 "" H 5950 2400 50  0001 C CNN
+	1    5950 2400
+	1    0    0    -1
+$EndComp
+Wire Wire Line
+	5950 1600 5950 1700
+Wire Wire Line
+	5950 1200 5950 1300
 $Comp
 L Device:R_Small R5
 U 1 1 5E08A9F3
-P 6850 1800
-F 0 "R5" H 6880 1820 50  0000 L CNN
-F 1 "1k" H 6880 1760 50  0000 L CNN
-F 2 "KiCad/Resistor_SMD.pretty:R_0603_1608Metric" H 6850 1800 50  0001 C CNN
-F 3 "" H 6850 1800 50  0001 C CNN
-	1    6850 1800
+P 5950 1800
+F 0 "R5" H 5980 1820 50  0000 L CNN
+F 1 "1k" H 5980 1760 50  0000 L CNN
+F 2 "KiCad/Resistor_SMD.pretty:R_0603_1608Metric" H 5950 1800 50  0001 C CNN
+F 3 "" H 5950 1800 50  0001 C CNN
+	1    5950 1800
 	1    0    0    -1
 $EndComp
@@
 L Device:LED D3
 U 1 1 5E08A9F2
-P 6850 1450
-F 0 "D3" H 6850 1550 50  0000 C CNN
-F 1 "PWR" H 6850 1350 50  0000 C CNN
-F 2 "KiCad/LED_SMD.pretty:LED_0603_1608Metric" H 6850 1450 50  0001 C CNN
-F 3 "http://www.kingbrightusa.com/images/catalog/SPEC/APT1608LZGCK.pdf" H 6850 1450 50  0001 C CNN
-F 4 "Kingbright" H 6850 1450 60  0001 C CNN "MFN"
-F 5 "APT1608LZGCK" H 6850 1450 60  0001 C CNN "MFP"
-F 6 "Green 525nm LED Indication - Discrete 2.65V 2mA 0603 (1608 Metric)" H 6850 1450 60  0001 C CNN "Description"
-F 7 "Green" H 6850 1450 50  0001 C CNN "Characteristics"
-F 8 "Digikey" H 6850 1450 50  0001 C CNN "Vendor"
-F 9 "754-1934-1-ND " H 6850 1450 50  0001 C CNN "SKU"
-	1    6850 1450
+P 5950 1450
+F 0 "D3" H 5950 1550 50  0000 C CNN
+F 1 "PWR" H 5950 1350 50  0000 C CNN
+F 2 "KiCad/LED_SMD.pretty:LED_0603_1608Metric" H 5950 1450 50  0001 C CNN
+F 3 "http://www.kingbrightusa.com/images/catalog/SPEC/APT1608LZGCK.pdf" H 5950 1450 50  0001 C CNN
+F 4 "Kingbright" H 5950 1450 60  0001 C CNN "MFN"
+F 5 "APT1608LZGCK" H 5950 1450 60  0001 C CNN "MFP"
+F 6 "Green 525nm LED Indication - Discrete 2.65V 2mA 0603 (1608 Metric)" H 5950 1450 60  0001 C CNN "Description"
+F 7 "Green" H 5950 1450 50  0001 C CNN "Characteristics"
+F 8 "Digikey" H 5950 1450 50  0001 C CNN "Vendor"
+F 9 "754-1934-1-ND " H 5950 1450 50  0001 C CNN "SKU"
+	1    5950 1450
 	0    -1   -1   0
 $EndComp
@@
 L power:+5V #PWR03
 U 1 1 5E1A2521
-P 5500 1200
-F 0 "#PWR03" H 5500 1050 50  0001 C CNN
-F 1 "+5V" H 5515 1373 50  0000 C CNN
-F 2 "" H 5500 1200 50  0001 C CNN
-F 3 "" H 5500 1200 50  0001 C CNN
-	1    5500 1200
+P 5375 1200
+F 0 "#PWR03" H 5375 1050 50  0001 C CNN
+F 1 "+5V" H 5390 1373 50  0000 C CNN
+F 2 "" H 5375 1200 50  0001 C CNN
+F 3 "" H 5375 1200 50  0001 C CNN
+	1    5375 1200
 	1    0    0    -1
 $EndComp
@@
 L power:+5V #PWR04
 U 1 1 5E1A2EA6
-P 6850 1200
-F 0 "#PWR04" H 6850 1050 50  0001 C CNN
-F 1 "+5V" H 6865 1373 50  0000 C CNN
-F 2 "" H 6850 1200 50  0001 C CNN
-F 3 "" H 6850 1200 50  0001 C CNN
-	1    6850 1200
+P 5950 1200
+F 0 "#PWR04" H 5950 1050 50  0001 C CNN
+F 1 "+5V" H 5965 1373 50  0000 C CNN
+F 2 "" H 5950 1200 50  0001 C CNN
+F 3 "" H 5950 1200 50  0001 C CNN
+	1    5950 1200
 	1    0    0    -1
 $EndComp
@@
 Text Label 3175 1700 2    50   ~ 0
 VIN
-Text Notes 2975 1550 0    50   Italic 0
+Text Notes 2875 1550 0    50   Italic 0
 5-16 V
 Wire Wire Line
@@
 Wire Wire Line
 	3850 1700 4050 1700
-$Comp
-L power:PWR_FLAG #FLG0104
-U 1 1 5E22F9C4
-P 8950 4100
-F 0 "#FLG0104" H 8950 4175 50  0001 C CNN
-F 1 "PWR_FLAG" H 8950 4274 50  0001 C CNN
-F 2 "" H 8950 4100 50  0001 C CNN
-F 3 "~" H 8950 4100 50  0001 C CNN
-	1    8950 4100
-	1    0    0    -1
-$EndComp
-Connection ~ 8950 4100
-Wire Wire Line
-	5500 1200 5500 1700
+Wire Wire Line
+	5375 1200 5375 1700
 $Comp
 L power:PWR_FLAG #FLG0101
@@
 $EndComp
 Wire Wire Line
-	3175 1700 3650 1700
-Connection ~ 3650 1700
-Wire Wire Line
 	9200 2300 9450 2300
 Wire Wire Line
@@
 FC_RX
 $Comp
-L Jumper:SolderJumper_2_Bridged JP3
+L Jumper:SolderJumper_2_Open JP3
 U 1 1 5E2A57BA
 P 4450 4200
 F 0 "JP3" H 4575 4250 50  0000 C CNN
 F 1 "INT" H 4450 4314 50  0001 C CNN
-F 2 "KiCad/Jumper.pretty:SolderJumper-2_P1.3mm_Bridged_RoundedPad1.0x1.5mm" H 4450 4200 50  0001 C CNN
+F 2 "KiCad/Jumper.pretty:SolderJumper-2_P1.3mm_Open_RoundedPad1.0x1.5mm" H 4450 4200 50  0001 C CNN
 F 3 "~" H 4450 4200 50  0001 C CNN
 F 4 "nofit" H 4450 4200 50  0001 C CNN "Config"
@@
 $EndComp
 $Comp
-L Jumper:SolderJumper_2_Bridged JP4
+L Jumper:SolderJumper_2_Open JP4
 U 1 1 5E2BEBB3
 P 4450 4350
 F 0 "JP4" H 4575 4400 50  0000 C CNN
 F 1 "INT" H 4450 4464 50  0001 C CNN
-F 2 "KiCad/Jumper.pretty:SolderJumper-2_P1.3mm_Bridged_RoundedPad1.0x1.5mm" H 4450 4350 50  0001 C CNN
+F 2 "KiCad/Jumper.pretty:SolderJumper-2_P1.3mm_Open_RoundedPad1.0x1.5mm" H 4450 4350 50  0001 C CNN
 F 3 "~" H 4450 4350 50  0001 C CNN
 F 4 "nofit" H 4450 4350 50  0001 C CNN "Config"
@@
 	1    0    0    -1
 $EndComp
+$Comp
+L power:+BATT #PWR0117
+U 1 1 5E29B53C
+P 8950 4100
+F 0 "#PWR0117" H 8950 3950 50  0001 C CNN
+F 1 "+BATT" H 8925 4250 50  0000 C CNN
+F 2 "" H 8950 4100 50  0001 C CNN
+F 3 "" H 8950 4100 50  0001 C CNN
+	1    8950 4100
+	1    0    0    -1
+$EndComp
+Connection ~ 8950 4100
+$Comp
+L Connector:TestPoint TP1
+U 1 1 5E29D75D
+P 9975 4100
+F 0 "TP1" H 9917 4126 50  0000 R CNN
+F 1 "RTC_BAT" H 9917 4217 50  0000 R CNN
+F 2 "KiCad/TestPoint.pretty:TestPoint_Pad_D2.5mm" H 10175 4100 50  0001 C CNN
+F 3 "~" H 10175 4100 50  0001 C CNN
+F 4 "nofit" H 9975 4100 50  0001 C CNN "Config"
+	1    9975 4100
+	-1   0    0    1
+$EndComp
+$Comp
+L power:+BATT #PWR0119
+U 1 1 5E29EF81
+P 9975 4100
+F 0 "#PWR0119" H 9975 3950 50  0001 C CNN
+F 1 "+BATT" H 9950 4250 50  0000 C CNN
+F 2 "" H 9975 4100 50  0001 C CNN
+F 3 "" H 9975 4100 50  0001 C CNN
+	1    9975 4100
+	1    0    0    -1
+$EndComp
+$Comp
+L Device:R_Small R1
+U 1 1 5E14102C
+P 2100 5550
+F 0 "R1" H 2130 5570 50  0000 L CNN
+F 1 "120R" H 2130 5510 50  0000 L CNN
+F 2 "KiCad/Resistor_SMD.pretty:R_0603_1608Metric" H 2100 5550 50  0001 C CNN
+F 3 "" H 2100 5550 50  0001 C CNN
+F 4 "Rterm" H 1950 5550 50  0000 C CNN "Description"
+F 5 "1%" H 2100 5550 50  0001 C CNN "Characteristics"
+	1    2100 5550
+	1    0    0    -1
+$EndComp
+Connection ~ 5050 1700
+Wire Wire Line
+	4650 1700 5050 1700
+Wire Wire Line
+	5050 2200 5050 2400
+Wire Wire Line
+	5050 1700 5050 1900
+$Comp
+L Device:C C2
+U 1 1 5DA6480B
+P 5050 2050
+F 0 "C2" H 5165 2096 50  0000 L CNN
+F 1 "1uF" H 5165 2005 50  0000 L CNN
+F 2 "KiCad/Capacitor_SMD.pretty:C_0603_1608Metric" H 5088 1900 50  0001 C CNN
+F 3 "~" H 5050 2050 50  0001 C CNN
+F 4 "X5R 20V" H 5050 2050 50  0001 C CNN "Characteristics"
+	1    5050 2050
+	1    0    0    -1
+$EndComp
+$Comp
+L power:GND #PWR0103
+U 1 1 5E08A9F1
+P 5050 2400
+F 0 "#PWR0103" H 5050 2150 50  0001 C CNN
+F 1 "GND" H 5050 2250 50  0000 C CNN
+F 2 "" H 5050 2400 50  0001 C CNN
+F 3 "" H 5050 2400 50  0001 C CNN
+	1    5050 2400
+	1    0    0    -1
+$EndComp
+Connection ~ 3650 1700
+Wire Wire Line
+	5050 1700 5375 1700
+$Comp
+L Device:D_Small D4
+U 1 1 5E343F8B
+P 3400 1700
+F 0 "D4" H 3350 1600 50  0000 L CNN
+F 1 "40V 200mA" H 3160 1600 50  0001 L CNN
+F 2 "KiCad/Diode_SMD.pretty:D_0603_1608Metric" V 3400 1700 50  0001 C CNN
+F 3 "~" V 3400 1700 50  0001 C CNN
+F 4 "Diode Schottky 40V 200mA (DC) Surface Mount 0603 (1608 Metric)" H 3400 1700 50  0001 C CNN "Description"
+F 5 "AVX Corporation" H 3400 1700 50  0001 C CNN "MFN"
+F 6 "SD0603S040S0R2" H 3400 1700 50  0001 C CNN "MFP"
+F 7 "478-7798-1-ND" H 3400 1700 50  0001 C CNN "SKU"
+F 8 "Digikey" H 3400 1700 50  0001 C CNN "Vendor"
+F 9 "Don't allow back powering bus and reverse polarity protect" H 3400 1700 50  0001 C CNN "Notes"
+F 10 "40V 200mA" H 3400 1700 50  0001 C CNN "Characteristics"
+	1    3400 1700
+	-1   0    0    1
+$EndComp
+Wire Wire Line
+	3175 1700 3300 1700
+Wire Wire Line
+	3500 1700 3650 1700
+Text Notes 2380 1180 0    50   ~ 0
+250 mA! 10k charge current resistor on Feather if using LiPo = 100 mA
 $EndSCHEMATC

Commit message: correct MFP/MPN and add kitspace tsv
Parts:
- BT1: MFP BAT-HLD-012-SMT-TR -> (none); MPN (none) -> BAT-HLD-012-SMT-TR
- D1, D2: MFP APT1608LSECK/J4-PRV -> (none); MPN (none) -> APT1608LSECK/J4-PRV
- D3: MFP APT1608LZGCK -> (none); MPN (none) -> APT1608LZGCK
- D4: MFP SD0603S040S0R2 -> (none); MPN (none) -> SD0603S040S0R2
- J4: MFP 53261-0471 -> (none); MPN (none) -> 53261-0471
- U1: MFP DS3231MZ+ -> (none); MPN (none) -> DS3231MZ+
- U2: MFP MCP2515T-I/ST -> (none); MPN (none) -> MCP2515T-I/ST
- U3: MFP MCP2551-I/SN -> (none); MPN (none) -> MCP2551-I/SN
- U4: MFP MCP1703T-5002E/CB -> (none); MPN (none) -> MCP1703T-5002E/CB
- Y1: MFP TSX-3225 16.0000MF18X-AC0 -> (none); MPN (none) -> TSX-3225 16.0000MF18X-AC0
Changed lines of the file:
@@
 F 3 "http://ww1.microchip.com/downloads/en/devicedoc/21667d.pdf" H 2800 4950 50  0001 C CNN
 F 4 "Microchip Technology" H 2800 4950 50  0001 C CNN "MFN"
-F 5 "MCP2551-I/SN" H 2800 4950 50  0001 C CNN "MFP"
+F 5 "MCP2551-I/SN" H 2800 4950 50  0001 C CNN "MPN"
 F 6 "3.3 V 250 mA upto 16 V input" H 2800 4950 50  0001 C CNN "Description"
 F 7 "Digikey" H 2800 4950 50  0001 C CNN "Vendor"
@@
 F 3 "http://datasheets.maximintegrated.com/en/ds/DS3231M.pdf" H 9050 4200 50  0001 C CNN
 F 4 "Maxim" H 9050 4800 50  0001 C CNN "MFN"
-F 5 "DS3231MZ+" H 9050 4800 50  0001 C CNN "MFP"
+F 5 "DS3231MZ+" H 9050 4800 50  0001 C CNN "MPN"
 F 6 "Digikey" H 9050 4800 50  0001 C CNN "Vendor"
 F 7 "DS3231MZ+-ND " H 9050 4800 50  0001 C CNN "SKU"
@@
 F 3 "~" V 8550 4160 50  0001 C CNN
 F 4 "Linx Technologies" H 8550 4100 50  0001 C CNN "MFN"
-F 5 "BAT-HLD-012-SMT-TR" H 8550 4100 50  0001 C CNN "MFP"
+F 5 "BAT-HLD-012-SMT-TR" H 8550 4100 50  0001 C CNN "MPN"
 F 6 "Digikey" H 8550 4100 50  0001 C CNN "Vendor"
 F 7 "BAT-HLD-012-SMTCT-ND" H 8550 4100 50  0001 C CNN "SKU"
@@
 F 3 "http://www.microchip.com/mymicrochip/filehandler.aspx?ddocname=en530937" H 4350 1650 50  0001 C CNN
 F 4 "Microchip Technology" H 4350 1700 60  0001 C CNN "MFN"
-F 5 "MCP1703T-5002E/CB" H 4350 1700 60  0001 C CNN "MFP"
+F 5 "MCP1703T-5002E/CB" H 4350 1700 60  0001 C CNN "MPN"
 F 6 "5 V LDO" H 4350 1700 60  0001 C CNN "Description"
 F 7 "Digikey" H 4350 1700 50  0001 C CNN "Vendor"
@@
 F 3 "http://ww1.microchip.com/downloads/en/DeviceDoc/MCP2515-Stand-Alone-CAN-Controller-with-SPI-20001801J.pdf" H 5500 4650 50  0001 C CNN
 F 4 "Microchip Technology" H 5400 5450 50  0001 C CNN "MFN"
-F 5 "MCP2515T-I/ST" H 5400 5450 50  0001 C CNN "MFP"
+F 5 "MCP2515T-I/ST" H 5400 5450 50  0001 C CNN "MPN"
 F 6 "MCP2515T-I/STCT-ND" H 5400 5450 50  0001 C CNN "SKU"
 F 7 "Digikey" H 5400 5450 50  0001 C CNN "Vendor"
@@
 F 3 "http://www.kingbrightusa.com/images/catalog/SPEC/APT1608LSECK-J4-PRV.pdf" H 3850 3950 50  0001 C CNN
 F 4 "Kingbright" H 3850 3950 60  0001 C CNN "MFN"
-F 5 "APT1608LSECK/J4-PRV " H 3850 3950 60  0001 C CNN "MFP"
+F 5 "APT1608LSECK/J4-PRV " H 3850 3950 60  0001 C CNN "MPN"
 F 6 "Orange 605nm LED Indication - Discrete 1.8V 2mA 0603 (1608 Metric) " H 3850 3950 60  0001 C CNN "Description"
 F 7 "Orange" H 3850 3950 50  0001 C CNN "Characteristics"
@@
 F 3 "http://www.kingbrightusa.com/images/catalog/SPEC/APT1608LSECK-J4-PRV.pdf" H 3500 3950 50  0001 C CNN
 F 4 "Kingbright" H 3500 3950 60  0001 C CNN "MFN"
-F 5 "APT1608LSECK/J4-PRV " H 3500 3950 60  0001 C CNN "MFP"
+F 5 "APT1608LSECK/J4-PRV " H 3500 3950 60  0001 C CNN "MPN"
 F 6 "Orange 605nm LED Indication - Discrete 1.8V 2mA 0603 (1608 Metric)" H 3500 3950 60  0001 C CNN "Description"
 F 7 "Orange" H 3500 3950 50  0001 C CNN "Characteristics"
@@
 F 3 "http://www.kingbrightusa.com/images/catalog/SPEC/APT1608LZGCK.pdf" H 5950 1450 50  0001 C CNN
 F 4 "Kingbright" H 5950 1450 60  0001 C CNN "MFN"
-F 5 "APT1608LZGCK" H 5950 1450 60  0001 C CNN "MFP"
+F 5 "APT1608LZGCK" H 5950 1450 60  0001 C CNN "MPN"
 F 6 "Green 525nm LED Indication - Discrete 2.65V 2mA 0603 (1608 Metric)" H 5950 1450 60  0001 C CNN "Description"
 F 7 "Green" H 5950 1450 50  0001 C CNN "Characteristics"
@@
 F 3 "~" H 1400 2900 50  0001 C CNN
 F 4 "Molex" H 1400 2900 50  0001 C CNN "MFN"
-F 5 "53261-0471" H 1400 2900 50  0001 C CNN "MFP"
+F 5 "53261-0471" H 1400 2900 50  0001 C CNN "MPN"
 F 6 "Digikey" H 1400 2900 50  0001 C CNN "Vendor"
 F 7 "WM7622CT-ND" H 1400 2900 50  0001 C CNN "SKU"
@@
 F 4 "9pF" H 6550 5550 50  0001 C CNN "Description"
 F 5 "Epson" H 6550 5550 50  0001 C CNN "MFN"
-F 6 "TSX-3225 16.0000MF18X-AC0" H 6550 5550 50  0001 C CNN "MFP"
+F 6 "TSX-3225 16.0000MF18X-AC0" H 6550 5550 50  0001 C CNN "MPN"
 F 7 "SER4070CT-ND" H 6550 5550 50  0001 C CNN "SKU"
 F 8 "Digikey" H 6550 5550 50  0001 C CNN "Vendor"
@@
 F 4 "Diode Schottky 40V 200mA (DC) Surface Mount 0603 (1608 Metric)" H 3400 1700 50  0001 C CNN "Description"
 F 5 "AVX Corporation" H 3400 1700 50  0001 C CNN "MFN"
-F 6 "SD0603S040S0R2" H 3400 1700 50  0001 C CNN "MFP"
+F 6 "SD0603S040S0R2" H 3400 1700 50  0001 C CNN "MPN"
 F 7 "478-7798-1-ND" H 3400 1700 50  0001 C CNN "SKU"
 F 8 "Digikey" H 3400 1700 50  0001 C CNN "Vendor"
